File: beaglebone_gateway/v1/beaglebone_gateway_v1.kicad_sch (KiCad schematic)
At the start: 2 parts, among them P8 BeagleBone_Black_Header, P9 BeagleBone_Black_Header

Commit message: Remove comments, add sheets description
Other:
- sheet Devices: file beaglebone_gateway_vi_devices.kicad_sch -> beaglebone_gateway_v1_devices.kicad_sch
- note added: "Beaglebone Black LoRa gateway HAT."
- note added: "Beaglebone Black LoRa gateway HAT. Buzzverse. Authors: Jakub Martyński Maciej Wołosewicz"
- note removed: "BeagleBone Black Pin Modes: https://elinux.org/Beagleboard:Cape_Expansion_Headers Cape requirements are documented in the BeagleBone Black SRM: https://github.com/beagleboard/beaglebone-black/wiki/System-Reference-Manual"
- note removed: "Beaglebone - gateway (Jakub Martyński - Uniwersytet Zielonogórski)"
- note removed: "Może warto również dodać jakieś 2 przyciski do nieużywanych GPIO, co nam pozwoli sterować programem jak nie będzie np. podłączony komputer (to jest raczej nice to have i może być również zrobione w wersji 2)."
- note removed: "Ogólne: - Nie używaj symbolu omega (tak, to są ohmy ale nie używa się. Widać, że to jest rezystor więc wystarczy np. 1, 1k, 1M - Na koniec żeby ktoś kto nie ma KiCada mógł oglądać wygodnie schemat - zamiast robić screenshoty - "Wydrukuj do PDFa" - Schemat i PCB."
- note removed: "Podłącz piny DIO0-DIO5 do jakiś pinów na złączach. Mamy sporo wolnych a mogą się przydać do odczytywania dodatkowych informacji o układzie."
- note removed: "Zastanów się czy nie warto dodać jakiegoś switcha i podłączyć PWR_BUT i SYS_RESET. Jak nałożymy tą nakładkę na Beaglebone to stracimy dostęp (a przynajmniej bardzo go utrudnimy) do przycisków na płycie. (Nice to have i może być również zrobione w wersji 2 bo wydaje się proste do zrobienia)."
Changed lines of the file:
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@@
     (stroke (width 0) (type solid))
   )
-  (text "Beaglebone - gateway (Jakub Martyński - Uniwersytet Zielonogórski)"
-    (at 186.69 190.5 0)
+  (text "Beaglebone Black LoRa gateway HAT." (at 186.69 190.5 0)
     (effects (font (size 1.27 1.27) (color 9 0 241 1)) (justify left bottom))
   )
-  (text "BeagleBone Black Pin Modes:\nhttps://elinux.org/Beagleboard:Cape_Expansion_Headers\n\nCape requirements are documented in the BeagleBone Black SRM:\nhttps://github.com/beagleboard/beaglebone-black/wiki/System-Reference-Manual"
-    (at 177.8 180.34 0)
-    (effects (font (size 1.27 1.27)) (justify left bottom))
-  )
-  (text "Podłącz piny DIO0-DIO5 do jakiś pinów na złączach.\nMamy sporo wolnych a mogą się przydać do odczytywania\ndodatkowych informacji o układzie."
-    (at -1.27 -29.21 0)
-    (effects (font (size 1.27 1.27) (color 241 174 8 1)) (justify left bottom))
-  )
-  (text "Może warto również dodać jakieś 2 przyciski\ndo nieużywanych GPIO, co nam pozwoli sterować\nprogramem jak nie będzie np. podłączony\nkomputer (to jest raczej nice to have i może\nbyć również zrobione w wersji 2)."
-    (at 60.96 -22.86 0)
-    (effects (font (size 1.27 1.27) (color 241 174 8 1)) (justify left bottom))
-  )
-  (text "Ogólne:\n- Nie używaj symbolu omega (tak, to są ohmy ale nie używa\nsię. Widać, że to jest rezystor więc wystarczy np. 1, 1k, 1M\n- Na koniec żeby ktoś kto nie ma KiCada mógł oglądać wygodnie\nschemat - zamiast robić screenshoty - \"Wydrukuj do PDFa\" - Schemat i PCB.\n"
-    (at 121.92 -26.67 0)
-    (effects (font (size 1.27 1.27) (color 241 174 8 1)) (justify left bottom))
-  )
-  (text "Zastanów się czy nie warto dodać jakiegoś switcha\ni podłączyć PWR_BUT i SYS_RESET. Jak nałożymy tą nakładkę na\nBeaglebone to stracimy dostęp (a przynajmniej bardzo\ngo utrudnimy) do przycisków na płycie.\n\n(Nice to have i może\nbyć również zrobione w wersji 2\nbo wydaje się proste do zrobienia)."
-    (at -46.99 -7.62 0)
-    (effects (font (size 1.27 1.27) (color 241 174 8 1)) (justify left bottom))
+  (text "Beaglebone Black LoRa gateway HAT. Buzzverse.\n\nAuthors:\nJakub Martyński\nMaciej Wołosewicz"
+    (at 177.8 177.8 0)
+    (effects (font (size 1.27 1.27)) (justify left bottom))
   )
   (label "GPIO45" (at 175.26 68.58 0) (fields_autoplaced)
@@
       (effects (font (size 1.27 1.27)) (justify left bottom))
     )
-    (property "Sheetfile" "beaglebone_gateway_vi_devices.kicad_sch" (at 25.4 31.0646 0)
+    (property "Sheetfile" "beaglebone_gateway_v1_devices.kicad_sch" (at 25.4 31.0646 0)
       (effects (font (size 1.27 1.27)) (justify left top))
     )

Commit message: Add ADC divider cut off using complementary mosfet transistors
Parts:
- added TP4: GPIO23, TestPoint:TestPoint_Pad_D1.5mm, symbol Connector:TestPoint_Probe
- added TP5: GPIO47, TestPoint:TestPoint_Pad_D1.5mm, symbol Connector:TestPoint_Probe
- added TP6: GPIO27, TestPoint:TestPoint_Pad_D1.5mm, symbol Connector:TestPoint_Probe
- added TP7: GPIO22, TestPoint:TestPoint_Pad_D1.5mm, symbol Connector:TestPoint_Probe
- added TP8: PWR_BUT, TestPoint:TestPoint_Pad_D1.5mm, symbol Connector:TestPoint_Probe
Connections:
- net GPIO22: now also TP7.1
- net GPIO23: now also TP4.1
- net GPIO27: now also TP6.1
- net GPIO47: now also TP5.1
- net PWR_BUT: now also TP8.1
- net GPIO44 renamed BATT_CHARGE_CURRENT_ADC_EN
- net GPIO68 renamed BATT_VOLTAGE_ADC_EN
- no-connect marks 58 -> 51
Other:
- added sheet ADC (beaglebone_gateway_v1_adc.kicad_sch)
